File: BLE_WIFI_HID/BLE_WIFI_HID.kicad_pcb (KiCad board)
At the start: 2 copper layers, 62.9 x 33.4 mm, 25 parts, among them J1 Conn_02x03_Odd_Even, J2 Conn_02x03_Odd_Even, P3 PROGRAMMER SERIAL, P4 Battery, U1 ESP32-WROOM, U2 AP2112K-3.3TRG1, U3 MCP73831T-2ACI/OT

Commit message: Acomodo conectores
Parts:
- moved J1 1.23 mm to (148.6, 92.8)
- moved J2 0.23 mm to (205.5, 92.8)
Routing:
- net /ESP_GPIO0: track 89.1 -> 0.00 mm
- net /MOSI: track 61.6 -> 0.00 mm
Changed lines of the file:
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@@
   (general
     (thickness 1.6)
-    (drawings 5)
-    (tracks 83)
+    (drawings 8)
+    (tracks 61)
     (zones 0)
     (modules 25)
@@
   )
   (module Pines:62000621121 (layer F.Cu)
-    (at 149.808 92.833 270)
+    (at 148.575 92.85 270)
     (descr "WR-PHD 2.00mm Dual Pin Header, 6 Pins")
     (fp_text reference J1 (at -1.8864 -2.7633 270) (layer F.SilkS)
@@
   )
   (module Pines:62000621121 (layer F.Cu)
-    (at 205.508 93.033 270)
+    (at 205.5 92.8 270)
     (descr "WR-PHD 2.00mm Dual Pin Header, 6 Pins")
     (fp_text reference J2 (at -1.8864 -2.7633 270) (layer F.SilkS)
@@
       (xy -0.085266 -2.823537) (xy 0.064388 -2.823445)) (layer F.SilkS) (width 0.01))
   )
+  (dimension 60.975185 (width 0.15) (layer Margin)
+    (gr_text "60.975 mm" (at 177.102626 116.323736 0.1409487428) (layer Margin)
+      (effects (font (size 1 1) (thickness 0.15)))
+    )
+    (feature1 (pts (xy 207.525 89.775) (xy 207.588371 115.535159)))
+    (feature2 (pts (xy 146.55 89.925) (xy 146.613371 115.685159)))
+    (crossbar (pts (xy 146.611928 115.09874) (xy 207.586928 114.94874)))
+    (arrow1a (pts (xy 207.586928 114.94874) (xy 206.46187 115.53793)))
+    (arrow1b (pts (xy 207.586928 114.94874) (xy 206.458985 114.365092)))
+    (arrow2a (pts (xy 146.611928 115.09874) (xy 147.739871 115.682388)))
+    (arrow2b (pts (xy 146.611928 115.09874) (xy 147.736986 114.50955)))
+  )
+  (dimension 20.85 (width 0.15) (layer Margin)
+    (gr_text "20.850 mm" (at 138.575 100.3 270) (layer Margin)
+      (effects (font (size 1 1) (thickness 0.15)))
+    )
+    (feature1 (pts (xy 146.55 110.725) (xy 139.288579 110.725)))
+    (feature2 (pts (xy 146.55 89.875) (xy 139.288579 89.875)))
+    (crossbar (pts (xy 139.875 89.875) (xy 139.875 110.725)))
+    (arrow1a (pts (xy 139.875 110.725) (xy 139.288579 109.598496)))
+    (arrow1b (pts (xy 139.875 110.725) (xy 140.461421 109.598496)))
+    (arrow2a (pts (xy 139.875 89.875) (xy 139.288579 91.001504)))
+    (arrow2b (pts (xy 139.875 89.875) (xy 140.461421 91.001504)))
+  )
+  (dimension 20.85 (width 0.15) (layer Margin)
+    (gr_text "20.850 mm" (at 213.525 100.25 270) (layer Margin)
+      (effects (font (size 1 1) (thickness 0.15)))
+    )
+    (feature1 (pts (xy 207.55 110.675) (xy 212.811421 110.675)))
+    (feature2 (pts (xy 207.55 89.825) (xy 212.811421 89.825)))
+    (crossbar (pts (xy 212.225 89.825) (xy 212.225 110.675)))
+    (arrow1a (pts (xy 212.225 110.675) (xy 211.638579 109.548496)))
+    (arrow1b (pts (xy 212.225 110.675) (xy 212.811421 109.548496)))
+    (arrow2a (pts (xy 212.225 89.825) (xy 211.638579 90.951504)))
+    (arrow2b (pts (xy 212.225 89.825) (xy 212.811421 90.951504)))
+  )
   (gr_text "Backpack BLE" (at 195.453 83.82) (layer B.SilkS)
     (effects (font (size 1.5 1.5) (thickness 0.3)) (justify mirror))
@@
   (segment (start 166.588 104.162) (end 166.588 102.548) (width 0.3) (layer F.Cu) (net 7))
   (segment (start 166.232 104.518) (end 166.588 104.162) (width 0.3) (layer F.Cu) (net 7))
-  (segment (start 178.403 97.663) (end 176.162 97.663) (width 0.3) (layer F.Cu) (net 8))
-  (segment (start 176.162 97.663) (end 175.2 98.625) (width 0.3) (layer F.Cu) (net 8))
-  (segment (start 175.2 98.625) (end 175.2 107.9) (width 0.3) (layer F.Cu) (net 8))
-  (segment (start 175.2 107.9) (end 174.675 108.425) (width 0.3) (layer F.Cu) (net 8))
-  (segment (start 174.675 108.425) (end 153.225 108.425) (width 0.3) (layer F.Cu) (net 8))
-  (segment (start 153.225 108.425) (end 152.525 107.725) (width 0.3) (layer F.Cu) (net 8))
-  (segment (start 152.525 107.725) (end 152.525 88.925) (width 0.3) (layer F.Cu) (net 8))
-  (segment (start 152.525 88.925) (end 151.625 88.025) (width 0.3) (layer F.Cu) (net 8))
-  (segment (start 151.625 88.025) (end 149.025 88.025) (width 0.3) (layer F.Cu) (net 8))
-  (segment (start 148.808 88.242) (end 148.808 90.833) (width 0.3) (layer F.Cu) (net 8))
-  (segment (start 149.025 88.025) (end 148.808 88.242) (width 0.3) (layer F.Cu) (net 8))
   (segment (start 171.678 94.298) (end 171.4 94.576) (width 0.3) (layer F.Cu) (net 11))
   (segment (start 172.628 94.298) (end 171.678 94.298) (width 0.3) (layer F.Cu) (net 11))
@@
   (segment (start 161.658 96.942) (end 161.658 98.238) (width 0.3) (layer F.Cu) (net 14))
   (segment (start 162 96.6) (end 161.658 96.942) (width 0.3) (layer F.Cu) (net 14))
-  (segment (start 196.403 98.933) (end 203.033 98.933) (width 0.3) (layer F.Cu) (net 36))
-  (segment (start 203.338 99.238) (end 203.338 105.188) (width 0.3) (layer F.Cu) (net 36))
-  (segment (start 203.033 98.933) (end 203.338 99.238) (width 0.3) (layer F.Cu) (net 36))
-  (segment (start 196.403 98.933) (end 197.203 98.933) (width 0.3) (layer F.Cu) (net 36))
-  (segment (start 150.808 106.715122) (end 150.808 94.833) (width 0.3) (layer F.Cu) (net 36))
-  (segment (start 206.163 105.188) (end 206.625 105.65) (width 0.3) (layer F.Cu) (net 36))
-  (segment (start 203.338 105.188) (end 206.163 105.188) (width 0.3) (layer F.Cu) (net 36))
-  (segment (start 206.625 105.65) (end 206.625 108.575) (width 0.3) (layer F.Cu) (net 36))
-  (segment (start 206.625 108.575) (end 206.125 109.075) (width 0.3) (layer F.Cu) (net 36))
-  (segment (start 206.125 109.075) (end 153.167878 109.075) (width 0.3) (layer F.Cu) (net 36))
-  (segment (start 153.167878 109.075) (end 150.808 106.715122) (width 0.3) (layer F.Cu) (net 36))
   (segment (start 176.853 84.963) (end 175.691 86.125) (width 0.3) (layer F.Cu) (net 37))
   (segment (start 178.403 84.963) (end 176.853 84.963) (width 0.3) (layer F.Cu) (net 37))

Commit message: batt and reset
Parts:
- moved R5 0.20 mm to (158.3, 81.5)
- moved C2 0.15 mm to (158.3, 84.7)
Routing:
- net /ESP_RESET: track 13.1 -> 49.4 mm, vias 0 -> 1
- net +3V3: track 11.5 -> 36.7 mm
- net /IO25: track 0.00 -> 22.9 mm
- net VCC: track 0.00 -> 14.2 mm
- net Net-(R5-Pad1): track 0.00 -> 9.22 mm
- net Net-(D1-Pad2): track 0.03 -> 2.65 mm
Changed lines of the file:
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@@
     (thickness 1.6)
     (drawings 8)
-    (tracks 61)
+    (tracks 117)
     (zones 0)
     (modules 25)
@@
   )
   (module Resistors_SMD:R_0805_HandSoldering (layer F.Cu)
-    (at 158.208 81.708)
+    (at 158.3 81.525)
     (descr "Resistor SMD 0805, hand soldering")
     (tags "resistor 0805")
@@
   )
   (module Capacitors_SMD:C_0805_HandSoldering (layer F.Cu)
-    (at 158.178 84.688 180)
+    (at 158.325 84.65 180)
     (descr "Capacitor SMD 0805, hand soldering")
     (tags "capacitor 0805")
@@
   (gr_line (start 208.648 110.668) (end 145.718 110.698) (layer Edge.Cuts) (width 0.15))
   (gr_line (start 208.488 77.338) (end 208.648 110.668) (layer Edge.Cuts) (width 0.15))
-  (segment (start 175.6 85.45) (end 170.2 85.45) (width 0.3) (layer F.Cu) (net 1))
   (segment (start 169.918 85.168) (end 169.918 83.568) (width 0.3) (layer F.Cu) (net 1))
   (segment (start 170.2 85.45) (end 169.918 85.168) (width 0.3) (layer F.Cu) (net 1))
@@
   (segment (start 178.403 83.693) (end 176.332 83.693) (width 0.3) (layer F.Cu) (net 1))
   (segment (start 175.95 85.1) (end 175.6 85.45) (width 0.3) (layer F.Cu) (net 1))
+  (segment (start 164.883 81.283) (end 164.883 84.883) (width 0.3) (layer F.Cu) (net 1))
+  (segment (start 164.883 84.883) (end 165.45 85.45) (width 0.3) (layer F.Cu) (net 1))
+  (segment (start 175.6 85.45) (end 170.45 85.45) (width 0.3) (layer F.Cu) (net 1))
+  (segment (start 170.45 85.45) (end 170.2 85.45) (width 0.3) (layer F.Cu) (net 1))
+  (segment (start 169.7 85.386) (end 169.918 85.168) (width 0.3) (layer F.Cu) (net 1))
+  (segment (start 169.7 85.45) (end 169.7 85.386) (width 0.3) (layer F.Cu) (net 1))
+  (segment (start 169.7 85.45) (end 170.45 85.45) (width 0.3) (layer F.Cu) (net 1))
+  (segment (start 164.473 90.898) (end 165.738 90.898) (width 0.3) (layer F.Cu) (net 1))
+  (segment (start 163.25 89.675) (end 164.473 90.898) (width 0.3) (layer F.Cu) (net 1))
+  (segment (start 160.106 89.675) (end 163.25 89.675) (width 0.3) (layer F.Cu) (net 1))
+  (segment (start 158.618 90.538) (end 159.243 90.538) (width 0.3) (layer F.Cu) (net 1))
+  (segment (start 159.243 90.538) (end 160.106 89.675) (width 0.3) (layer F.Cu) (net 1))
+  (segment (start 166.663 90.898) (end 167.45 90.111) (width 0.3) (layer F.Cu) (net 1))
+  (segment (start 165.738 90.898) (end 166.663 90.898) (width 0.3) (layer F.Cu) (net 1))
+  (segment (start 167.45 85.65) (end 167.65 85.45) (width 0.3) (layer F.Cu) (net 1))
+  (segment (start 167.65 85.45) (end 169.7 85.45) (width 0.3) (layer F.Cu) (net 1))
+  (segment (start 167.45 85.45) (end 167.65 85.45) (width 0.3) (layer F.Cu) (net 1))
+  (segment (start 167.45 90.111) (end 167.45 85.775) (width 0.3) (layer F.Cu) (net 1))
+  (segment (start 167.45 85.775) (end 167.45 85.45) (width 0.3) (layer F.Cu) (net 1))
+  (segment (start 167.45 85.65) (end 167.25 85.45) (width 0.3) (layer F.Cu) (net 1))
+  (segment (start 167.45 85.775) (end 167.45 85.65) (width 0.3) (layer F.Cu) (net 1))
+  (segment (start 165.45 85.45) (end 167.25 85.45) (width 0.3) (layer F.Cu) (net 1))
+  (segment (start 167.25 85.45) (end 167.45 85.45) (width 0.3) (layer F.Cu) (net 1))
+  (segment (start 159.65 84.575) (end 159.575 84.65) (width 0.3) (layer F.Cu) (net 3))
+  (segment (start 159.65 81.525) (end 159.65 84.575) (width 0.3) (layer F.Cu) (net 3))
+  (segment (start 158.618 87.838) (end 158.618 86.682) (width 0.3) (layer F.Cu) (net 3))
+  (segment (start 159.575 85.725) (end 159.575 84.65) (width 0.3) (layer F.Cu) (net 3))
+  (segment (start 158.618 86.682) (end 159.575 85.725) (width 0.3) (layer F.Cu) (net 3))
+  (segment (start 162.238 88.318) (end 160.743 88.318) (width 0.3) (layer F.Cu) (net 3))
+  (segment (start 160.263 87.838) (end 158.618 87.838) (width 0.3) (layer F.Cu) (net 3))
+  (segment (start 160.743 88.318) (end 160.263 87.838) (width 0.3) (layer F.Cu) (net 3))
+  (segment (start 160.708 100.938) (end 160.708 102.442) (width 0.3) (layer F.Cu) (net 3))
+  (segment (start 160.468 102.682) (end 160.468 104.518) (width 0.3) (layer F.Cu) (net 3))
+  (segment (start 160.708 102.442) (end 160.468 102.682) (width 0.3) (layer F.Cu) (net 3))
   (segment (start 160.678 98.208) (end 160.708 98.238) (width 0.3) (layer F.Cu) (net 4))
   (segment (start 156.878 98.208) (end 160.678 98.208) (width 0.3) (layer F.Cu) (net 4))
@@
   (segment (start 162.727 94.323) (end 162.523 94.323) (width 0.3) (layer F.Cu) (net 4))
   (segment (start 184.408 106.018) (end 184.388 106.038) (width 0.3) (layer F.Cu) (net 5))
+  (segment (start 186.978 106.038) (end 186.998 106.018) (width 0.3) (layer F.Cu) (net 5))
+  (segment (start 184.388 106.038) (end 186.978 106.038) (width 0.3) (layer F.Cu) (net 5))
   (segment (start 163.168 104.518) (end 166.232 104.518) (width 0.3) (layer F.Cu) (net 7))
   (segment (start 166.588 104.162) (end 166.588 102.548) (width 0.3) (layer F.Cu) (net 7))
@@
   (segment (start 171.177 97.023) (end 170.028 97.023) (width 0.3) (layer F.Cu) (net 11))
   (segment (start 171.4 96.8) (end 171.177 97.023) (width 0.3) (layer F.Cu) (net 11))
+  (segment (start 156.093 87.838) (end 154.85 86.595) (width 0.3) (layer F.Cu) (net 12))
+  (segment (start 156.718 87.838) (end 156.093 87.838) (width 0.3) (layer F.Cu) (net 12))
+  (segment (start 154.85 86.595) (end 154.85 82.1) (width 0.3) (layer F.Cu) (net 12))
+  (segment (start 155.425 81.525) (end 156.95 81.525) (width 0.3) (layer F.Cu) (net 12))
+  (segment (start 154.85 82.1) (end 155.425 81.525) (width 0.3) (layer F.Cu) (net 12))
   (segment (start 168.928 102.638) (end 168 101.71) (width 0.3) (layer F.Cu) (net 13))
   (segment (start 169.878 102.638) (end 168.928 102.638) (width 0.3) (layer F.Cu) (net 13))
@@
   (segment (start 170.308 86.642) (end 170.308 90.948) (width 0.3) (layer F.Cu) (net 37))
   (segment (start 170.825 86.125) (end 170.308 86.642) (width 0.3) (layer F.Cu) (net 37))
+  (segment (start 193.178 103.985919) (end 194.238919 102.925) (width 0.3) (layer B.Cu) (net 37))
+  (segment (start 193.178 105.188) (end 193.178 103.985919) (width 0.3) (layer B.Cu) (net 37))
+  (segment (start 194.238919 102.925) (end 194.238919 85.738919) (width 0.3) (layer B.Cu) (net 37))
+  (via (at 182.125 84.625) (size 0.6) (drill 0.4) (layers F.Cu B.Cu) (net 37))
+  (segment (start 194.238919 85.738919) (end 193.125 84.625) (width 0.3) (layer B.Cu) (net 37))
+  (segment (start 193.125 84.625) (end 182.125 84.625) (width 0.3) (layer B.Cu) (net 37))
+  (segment (start 182.125 84.625) (end 181.3 84.625) (width 0.3) (layer F.Cu) (net 37))
+  (segment (start 180.962 84.963) (end 178.403 84.963) (width 0.3) (layer F.Cu) (net 37))
+  (segment (start 181.3 84.625) (end 180.962 84.963) (width 0.3) (layer F.Cu) (net 37))
   (segment (start 196.403 93.853) (end 200.197 93.853) (width 0.3) (layer F.Cu) (net 42))
   (segment (start 200.197 93.853) (end 201.35 92.7) (width 0.3) (layer F.Cu) (net 42))
@@
   (segment (start 170.992 81.283) (end 167.583 81.283) (width 0.3) (layer F.Cu) (net 42))
   (segment (start 171.992001 80.282999) (end 170.992 81.283) (width 0.3) (layer F.Cu) (net 42))
+  (segment (start 186.048 103.318) (end 185.591 103.775) (width 0.3) (layer F.Cu) (net 43))
+  (segment (start 186.998 103.318) (end 186.048 103.318) (width 0.3) (layer F.Cu) (net 43))
+  (segment (start 185.591 103.775) (end 177.475 103.775) (width 0.3) (layer F.Cu) (net 43))
+  (segment (start 177.475 103.775) (end 175.7 102) (width 0.3) (layer F.Cu) (net 43))
+  (segment (start 175.7 102) (end 175.7 94.175) (width 0.3) (layer F.Cu) (net 43))
+  (segment (start 176.022 93.853) (end 178.403 93.853) (width 0.3) (layer F.Cu) (net 43))
+  (segment (start 175.7 94.175) (end 176.022 93.853) (width 0.3) (layer F.Cu) (net 43))
   (zone (net 2) (net_name GND) (layer F.Cu) (hatch edge 0.508)
     (connect_pads (clearance 0.508))
