File: BLE_WIFI_HID/BLE_WIFI_HID.kicad_pcb (KiCad board)
At the start: 2 copper layers, 62.9 x 33.4 mm, 25 parts, among them J1 Conn_02x03_Odd_Even, J2 Conn_02x03_Odd_Even, P3 PROGRAMMER SERIAL, P4 Battery, U1 ESP32-WROOM, U2 AP2112K-3.3TRG1, U3 MCP73831T-2ACI/OT

Commit message: Change Esp
Parts:
- moved D1 9.13 mm to (174.1, 107.9)
- moved R3 9.12 mm to (178.1, 106.6)
- moved U1 3.04 mm to (188.0, 90.7)
- moved P3 1.49 mm to (203.4, 106.7)
Routing:
- net /ESP_CS: track 51.7 -> 0.00 mm
- net /ESP_RESET: track 49.4 -> 0.00 mm, vias 1 -> 0
- net /IO25: track 22.9 -> 0.00 mm
- net +3V3: track 36.7 -> 27.4 mm
Changed lines of the file:
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@@
     (thickness 1.6)
     (drawings 8)
-    (tracks 117)
+    (tracks 84)
     (zones 0)
     (modules 25)
@@
   )
   (module LEDs:LED_0805_HandSoldering (layer F.Cu)
-    (at 183.038 106.038)
+    (at 174.113 107.938)
     (descr "Resistor SMD 0805, hand soldering")
     (tags "resistor 0805")
@@
   )
   (module Pin_Headers:Pin_Header_Straight_1x06_Pitch2.54mm (layer F.Cu)
-    (at 203.338 105.188 270)
+    (at 203.37 106.675 270)
     (descr "Through hole straight pin header, 1x06, 2.54mm pitch, single row")
     (tags "Through hole pin header THT 1x06 2.54mm single row")
@@
   )
   (module ESP32-footprints-Lib:ESP32-WROOM (layer F.Cu)
-    (at 187.403 87.673 180)
+    (at 188 90.65 180)
     (fp_text reference U1 (at -11.557 9.017 180) (layer F.SilkS)
       (effects (font (size 1 1) (thickness 0.15)))
@@
   )
   (module Resistors_SMD:R_0805_HandSoldering (layer F.Cu)
-    (at 186.998 104.668 270)
+    (at 178.073 106.568 270)
     (descr "Resistor SMD 0805, hand soldering")
     (tags "resistor 0805")
@@
   (segment (start 169.918 85.168) (end 169.918 83.568) (width 0.3) (layer F.Cu) (net 1))
   (segment (start 170.2 85.45) (end 169.918 85.168) (width 0.3) (layer F.Cu) (net 1))
-  (segment (start 175.95 84.075) (end 175.95 85.1) (width 0.3) (layer F.Cu) (net 1))
-  (segment (start 176.332 83.693) (end 175.95 84.075) (width 0.3) (layer F.Cu) (net 1))
-  (segment (start 178.403 83.693) (end 176.332 83.693) (width 0.3) (layer F.Cu) (net 1))
-  (segment (start 175.95 85.1) (end 175.6 85.45) (width 0.3) (layer F.Cu) (net 1))
   (segment (start 164.883 81.283) (end 164.883 84.883) (width 0.3) (layer F.Cu) (net 1))
   (segment (start 164.883 84.883) (end 165.45 85.45) (width 0.3) (layer F.Cu) (net 1))
-  (segment (start 175.6 85.45) (end 170.45 85.45) (width 0.3) (layer F.Cu) (net 1))
   (segment (start 170.45 85.45) (end 170.2 85.45) (width 0.3) (layer F.Cu) (net 1))
   (segment (start 169.7 85.386) (end 169.918 85.168) (width 0.3) (layer F.Cu) (net 1))
@@
   (segment (start 170.028 94.323) (end 162.727 94.323) (width 0.3) (layer F.Cu) (net 4))
   (segment (start 162.727 94.323) (end 162.523 94.323) (width 0.3) (layer F.Cu) (net 4))
-  (segment (start 184.408 106.018) (end 184.388 106.038) (width 0.3) (layer F.Cu) (net 5))
-  (segment (start 186.978 106.038) (end 186.998 106.018) (width 0.3) (layer F.Cu) (net 5))
-  (segment (start 184.388 106.038) (end 186.978 106.038) (width 0.3) (layer F.Cu) (net 5))
+  (segment (start 175.483 107.918) (end 175.463 107.938) (width 0.3) (layer F.Cu) (net 5))
+  (segment (start 178.053 107.938) (end 178.073 107.918) (width 0.3) (layer F.Cu) (net 5))
+  (segment (start 175.463 107.938) (end 178.053 107.938) (width 0.3) (layer F.Cu) (net 5))
   (segment (start 163.168 104.518) (end 166.232 104.518) (width 0.3) (layer F.Cu) (net 7))
   (segment (start 166.588 104.162) (end 166.588 102.548) (width 0.3) (layer F.Cu) (net 7))
@@
   (segment (start 161.658 96.942) (end 161.658 98.238) (width 0.3) (layer F.Cu) (net 14))
   (segment (start 162 96.6) (end 161.658 96.942) (width 0.3) (layer F.Cu) (net 14))
-  (segment (start 176.853 84.963) (end 175.691 86.125) (width 0.3) (layer F.Cu) (net 37))
-  (segment (start 178.403 84.963) (end 176.853 84.963) (width 0.3) (layer F.Cu) (net 37))
-  (segment (start 175.691 86.125) (end 170.825 86.125) (width 0.3) (layer F.Cu) (net 37))
-  (segment (start 170.308 86.642) (end 170.308 90.948) (width 0.3) (layer F.Cu) (net 37))
-  (segment (start 170.825 86.125) (end 170.308 86.642) (width 0.3) (layer F.Cu) (net 37))
-  (segment (start 193.178 103.985919) (end 194.238919 102.925) (width 0.3) (layer B.Cu) (net 37))
-  (segment (start 193.178 105.188) (end 193.178 103.985919) (width 0.3) (layer B.Cu) (net 37))
-  (segment (start 194.238919 102.925) (end 194.238919 85.738919) (width 0.3) (layer B.Cu) (net 37))
-  (via (at 182.125 84.625) (size 0.6) (drill 0.4) (layers F.Cu B.Cu) (net 37))
-  (segment (start 194.238919 85.738919) (end 193.125 84.625) (width 0.3) (layer B.Cu) (net 37))
-  (segment (start 193.125 84.625) (end 182.125 84.625) (width 0.3) (layer B.Cu) (net 37))
-  (segment (start 182.125 84.625) (end 181.3 84.625) (width 0.3) (layer F.Cu) (net 37))
-  (segment (start 180.962 84.963) (end 178.403 84.963) (width 0.3) (layer F.Cu) (net 37))
-  (segment (start 181.3 84.625) (end 180.962 84.963) (width 0.3) (layer F.Cu) (net 37))
-  (segment (start 196.403 93.853) (end 200.197 93.853) (width 0.3) (layer F.Cu) (net 42))
-  (segment (start 200.197 93.853) (end 201.35 92.7) (width 0.3) (layer F.Cu) (net 42))
-  (segment (start 201.35 92.7) (end 201.35 80.875) (width 0.3) (layer F.Cu) (net 42))
-  (segment (start 200.757999 80.282999) (end 171.992001 80.282999) (width 0.3) (layer F.Cu) (net 42))
-  (segment (start 201.35 80.875) (end 200.757999 80.282999) (width 0.3) (layer F.Cu) (net 42))
-  (segment (start 170.992 81.283) (end 167.583 81.283) (width 0.3) (layer F.Cu) (net 42))
-  (segment (start 171.992001 80.282999) (end 170.992 81.283) (width 0.3) (layer F.Cu) (net 42))
-  (segment (start 186.048 103.318) (end 185.591 103.775) (width 0.3) (layer F.Cu) (net 43))
-  (segment (start 186.998 103.318) (end 186.048 103.318) (width 0.3) (layer F.Cu) (net 43))
-  (segment (start 185.591 103.775) (end 177.475 103.775) (width 0.3) (layer F.Cu) (net 43))
-  (segment (start 177.475 103.775) (end 175.7 102) (width 0.3) (layer F.Cu) (net 43))
-  (segment (start 175.7 102) (end 175.7 94.175) (width 0.3) (layer F.Cu) (net 43))
-  (segment (start 176.022 93.853) (end 178.403 93.853) (width 0.3) (layer F.Cu) (net 43))
-  (segment (start 175.7 94.175) (end 176.022 93.853) (width 0.3) (layer F.Cu) (net 43))
   (zone (net 2) (net_name GND) (layer F.Cu) (hatch edge 0.508)
     (connect_pads (clearance 0.508))
