File: BLE_WIFI_HID/BLE_WIFI_HID.kicad_pcb (KiCad board)
At the start: 2 copper layers, 62.9 x 33.4 mm, 25 parts, among them J1 Conn_02x03_Odd_Even, J2 Conn_02x03_Odd_Even, P3 PROGRAMMER SERIAL, P4 Battery, U1 ESP32-WROOM, U2 AP2112K-3.3TRG1, U3 MCP73831T-2ACI/OT

Commit message: Conn left
Parts:
- moved J2 0.58 mm to (204.9, 92.7)
- moved J1 0.41 mm to (149.0, 92.8)
Routing:
- net /SCK: track 0.00 -> 92.8 mm, vias 0 -> 2
- net /MISO: track 0.00 -> 87.7 mm, vias 0 -> 2
- net /ESP_GPIO0: track 0.00 -> 79.6 mm, vias 0 -> 2
- net /MOSI: track 0.00 -> 52.9 mm
- net /ESP_RESET: track 0.00 -> 21.3 mm, vias 0 -> 2
- net GND: track 0.00 -> 11.0 mm
- net VCC: track 14.2 -> 25.1 mm
- net /ESP_CS: track 0.00 -> 10.2 mm, vias 0 -> 1

Commit message: Conn rigth
Routing:
- net /ESP_BUSY: track 0.00 -> 77.5 mm, vias 0 -> 4
- net /ESP_TX: track 0.00 -> 36.0 mm, vias 0 -> 3
- net /ESP_RX: track 0.00 -> 26.3 mm, vias 0 -> 1
- net /ESP_RTS: track 0.00 -> 16.1 mm, vias 0 -> 2
Changed lines of the file:
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@@
     (thickness 1.6)
     (drawings 8)
-    (tracks 161)
+    (tracks 234)
     (zones 0)
     (modules 25)
@@
   (segment (start 204.5 109.825) (end 205.8 108.525) (width 0.3) (layer B.Cu) (net 10))
   (segment (start 205.8 108.525) (end 205.8 99.275) (width 0.3) (layer B.Cu) (net 10))
-  (segment (start 205.8 99.275) (end 205.8 98.775) (width 0.3) (layer F.Cu) (net 10))
-  (segment (start 202.585 95.56) (end 197 95.56) (width 0.3) (layer F.Cu) (net 10))
-  (segment (start 205.8 98.775) (end 202.585 95.56) (width 0.3) (layer F.Cu) (net 10))
+  (segment (start 205.8 99.275) (end 205.8 98.325) (width 0.3) (layer F.Cu) (net 10))
+  (segment (start 205.8 98.325) (end 203.475 96) (width 0.3) (layer F.Cu) (net 10))
+  (segment (start 203.475 96) (end 199.4 96) (width 0.3) (layer F.Cu) (net 10))
+  (segment (start 198.96 95.56) (end 197 95.56) (width 0.3) (layer F.Cu) (net 10))
+  (segment (start 199.4 96) (end 198.96 95.56) (width 0.3) (layer F.Cu) (net 10))
   (segment (start 171.678 94.298) (end 171.4 94.576) (width 0.3) (layer F.Cu) (net 11))
   (segment (start 172.628 94.298) (end 171.678 94.298) (width 0.3) (layer F.Cu) (net 11))
@@
   (segment (start 167.7 92.225736) (end 168.977736 90.948) (width 0.3) (layer F.Cu) (net 37))
   (segment (start 167.7 92.65) (end 167.7 92.225736) (width 0.3) (layer F.Cu) (net 37))
-  (segment (start 203.000105 92.725) (end 201.475 94.250105) (width 0.3) (layer B.Cu) (net 42))
-  (segment (start 203.925 92.725) (end 203.000105 92.725) (width 0.3) (layer B.Cu) (net 42))
+  (via (at 204.9 89) (size 0.6) (drill 0.4) (layers F.Cu B.Cu) (net 38))
+  (segment (start 205.925 90.725) (end 205.925 90.025) (width 0.3) (layer F.Cu) (net 38))
+  (segment (start 205.925 90.025) (end 204.9 89) (width 0.3) (layer F.Cu) (net 38))
+  (segment (start 204.9 89) (end 202.5 89) (width 0.3) (layer B.Cu) (net 38))
+  (segment (start 202.5 89) (end 201.35 90.15) (width 0.3) (layer B.Cu) (net 38))
+  (segment (start 201.35 90.15) (end 201.35 92.625) (width 0.3) (layer B.Cu) (net 38))
+  (segment (start 201.35 92.625) (end 201.35 93.075) (width 0.3) (layer B.Cu) (net 38))
+  (segment (start 201.35 93.075) (end 201.35 93.425) (width 0.3) (layer B.Cu) (net 38))
+  (via (at 201.35 95.3) (size 0.6) (drill 0.4) (layers F.Cu B.Cu) (net 38))
+  (segment (start 201.35 93.425) (end 201.35 95.3) (width 0.3) (layer B.Cu) (net 38))
+  (segment (start 201.35 95.3) (end 200.125 95.3) (width 0.3) (layer F.Cu) (net 38))
+  (segment (start 199.115 94.29) (end 197 94.29) (width 0.3) (layer F.Cu) (net 38))
+  (segment (start 200.125 95.3) (end 199.115 94.29) (width 0.3) (layer F.Cu) (net 38))
+  (via (at 207.45 93.525) (size 0.6) (drill 0.4) (layers F.Cu B.Cu) (net 39))
+  (segment (start 174.65 96.65) (end 175.4 95.9) (width 0.3) (layer B.Cu) (net 39))
+  (via (at 175.4 95.9) (size 0.6) (drill 0.4) (layers F.Cu B.Cu) (net 39))
+  (segment (start 174.65 103.25) (end 174.65 96.65) (width 0.3) (layer B.Cu) (net 39))
+  (segment (start 173.575 104.325) (end 174.65 103.25) (width 0.3) (layer B.Cu) (net 39))
+  (segment (start 170.975 104.325) (end 173.575 104.325) (width 0.3) (layer B.Cu) (net 39))
+  (segment (start 169.3 106) (end 170.975 104.325) (width 0.3) (layer B.Cu) (net 39))
+  (segment (start 169.3 107.175) (end 169.3 106) (width 0.3) (layer B.Cu) (net 39))
+  (via (at 169.3 107.175) (size 0.6) (drill 0.4) (layers F.Cu B.Cu) (net 39))
+  (segment (start 169.3 109.7) (end 169.3 107.175) (width 0.3) (layer F.Cu) (net 39))
+  (segment (start 169.725 110.125) (end 169.3 109.7) (width 0.3) (layer F.Cu) (net 39))
+  (segment (start 170.525 110.125) (end 169.725 110.125) (width 0.3) (layer F.Cu) (net 39))
+  (segment (start 205.475736 110.125) (end 170.525 110.125) (width 0.3) (layer F.Cu) (net 39))
+  (segment (start 206.75 109.275) (end 206.325736 109.275) (width 0.3) (layer F.Cu) (net 39))
+  (segment (start 206.325736 109.275) (end 205.475736 110.125) (width 0.3) (layer F.Cu) (net 39))
+  (segment (start 207.45 108.575) (end 206.75 109.275) (width 0.3) (layer B.Cu) (net 39))
+  (segment (start 207.45 93.525) (end 207.45 108.575) (width 0.3) (layer B.Cu) (net 39))
+  (via (at 206.75 109.275) (size 0.6) (drill 0.4) (layers F.Cu B.Cu) (net 39))
+  (segment (start 206.65 92.725) (end 207.45 93.525) (width 0.3) (layer F.Cu) (net 39))
+  (segment (start 205.925 92.725) (end 206.65 92.725) (width 0.3) (layer F.Cu) (net 39))
+  (segment (start 175.74 95.56) (end 175.4 95.9) (width 0.3) (layer F.Cu) (net 39))
+  (segment (start 179 95.56) (end 175.74 95.56) (width 0.3) (layer F.Cu) (net 39))
+  (segment (start 205.925 95.649895) (end 204.9 96.674895) (width 0.3) (layer B.Cu) (net 40))
+  (segment (start 205.925 94.725) (end 205.925 95.649895) (width 0.3) (layer B.Cu) (net 40))
+  (segment (start 204.9 96.674895) (end 204.9 104.275) (width 0.3) (layer B.Cu) (net 40))
+  (via (at 200.825 104.875) (size 0.6) (drill 0.4) (layers F.Cu B.Cu) (net 40))
+  (segment (start 204.9 104.275) (end 204.3 104.875) (width 0.3) (layer B.Cu) (net 40))
+  (segment (start 204.3 104.875) (end 200.825 104.875) (width 0.3) (layer B.Cu) (net 40))
+  (segment (start 200.825 106.67) (end 200.83 106.675) (width 0.3) (layer F.Cu) (net 40))
+  (segment (start 200.825 104.875) (end 200.825 106.67) (width 0.3) (layer F.Cu) (net 40))
+  (segment (start 201.975 88.2) (end 200.965 89.21) (width 0.3) (layer F.Cu) (net 40))
+  (segment (start 200.965 89.21) (end 197 89.21) (width 0.3) (layer F.Cu) (net 40))
+  (segment (start 202.075 88.1) (end 201.975 88.2) (width 0.3) (layer B.Cu) (net 40))
+  (segment (start 205.425 88.1) (end 202.075 88.1) (width 0.3) (layer B.Cu) (net 40))
+  (via (at 201.975 88.2) (size 0.6) (drill 0.4) (layers F.Cu B.Cu) (net 40))
+  (via (at 205.425 88.1) (size 0.6) (drill 0.4) (layers F.Cu B.Cu) (net 40))
+  (segment (start 206.849895 94.725) (end 206.974895 94.85) (width 0.3) (layer F.Cu) (net 40))
+  (segment (start 205.925 94.725) (end 206.849895 94.725) (width 0.3) (layer F.Cu) (net 40))
+  (segment (start 206.974895 94.85) (end 207.5 94.85) (width 0.3) (layer F.Cu) (net 40))
+  (segment (start 207.5 94.85) (end 208.143959 94.206041) (width 0.3) (layer F.Cu) (net 40))
+  (segment (start 207.55965 88.1) (end 208.117325 88.657675) (width 0.3) (layer F.Cu) (net 40))
+  (segment (start 205.425 88.1) (end 207.55965 88.1) (width 0.3) (layer F.Cu) (net 40))
+  (segment (start 208.143959 94.206041) (end 208.117325 88.657675) (width 0.3) (layer F.Cu) (net 40))
+  (segment (start 203.925 94.725) (end 203.925 103.375) (width 0.3) (layer B.Cu) (net 41))
+  (via (at 199.75 104) (size 0.6) (drill 0.4) (layers F.Cu B.Cu) (net 41))
+  (segment (start 203.925 103.375) (end 203.3 104) (width 0.3) (layer B.Cu) (net 41))
+  (segment (start 203.3 104) (end 199.75 104) (width 0.3) (layer B.Cu) (net 41))
+  (segment (start 199.75 104) (end 198.85 104) (width 0.3) (layer F.Cu) (net 41))
+  (segment (start 198.29 104.56) (end 198.29 106.675) (width 0.3) (layer F.Cu) (net 41))
+  (segment (start 198.85 104) (end 198.29 104.56) (width 0.3) (layer F.Cu) (net 41))
+  (segment (start 203.925 94.725) (end 202.2 94.725) (width 0.3) (layer F.Cu) (net 41))
+  (segment (start 202.2 94.725) (end 200.2 92.725) (width 0.3) (layer F.Cu) (net 41))
+  (segment (start 200.2 92.725) (end 200.2 91.475) (width 0.3) (layer F.Cu) (net 41))
+  (segment (start 199.205 90.48) (end 197 90.48) (width 0.3) (layer F.Cu) (net 41))
+  (segment (start 200.2 91.475) (end 199.205 90.48) (width 0.3) (layer F.Cu) (net 41))
   (via (at 201.4 96.875) (size 0.6) (drill 0.4) (layers F.Cu B.Cu) (net 42))
-  (segment (start 201.475 94.250105) (end 201.475 96.8) (width 0.3) (layer B.Cu) (net 42))
   (segment (start 201.475 96.8) (end 201.4 96.875) (width 0.3) (layer B.Cu) (net 42))
   (segment (start 197.045 96.875) (end 197 96.83) (width 0.3) (layer F.Cu) (net 42))
   (segment (start 201.4 96.875) (end 197.045 96.875) (width 0.3) (layer F.Cu) (net 42))
+  (segment (start 201.824264 96.875) (end 202.775 95.924264) (width 0.3) (layer B.Cu) (net 42))
+  (segment (start 201.4 96.875) (end 201.824264 96.875) (width 0.3) (layer B.Cu) (net 42))
+  (segment (start 202.775 95.924264) (end 202.775 93.175) (width 0.3) (layer B.Cu) (net 42))
+  (segment (start 202.775 93.175) (end 203.3 92.65) (width 0.3) (layer B.Cu) (net 42))
+  (segment (start 203.85 92.65) (end 203.925 92.725) (width 0.3) (layer B.Cu) (net 42))
+  (segment (start 203.3 92.65) (end 203.85 92.65) (width 0.3) (layer B.Cu) (net 42))
   (zone (net 2) (net_name GND) (layer F.Cu) (hatch edge 0.508)
     (connect_pads (clearance 0.508))
     (min_thickness 0.254)
-    (fill (arc_segments 32) (thermal_gap 0.508) (thermal_bridge_width 0.508))
+    (fill yes (arc_segments 32) (thermal_gap 0.508) (thermal_bridge_width 0.508))
     (polygon
       (pts
@@
     (connect_pads (clearance 0.508))
     (min_thickness 0.254)
-    (fill (arc_segments 32) (thermal_gap 0.508) (thermal_bridge_width 0.508))
+    (fill yes (arc_segments 32) (thermal_gap 0.508) (thermal_bridge_width 0.508))
     (polygon
       (pts

Commit message: re-routeo
Parts:
- moved J1 55.9 mm to (204.9, 92.7)
- moved J2 55.9 mm to (149.1, 92.8)
- moved D1 4.15 mm to (170.0, 107.4)
- moved R3 1.61 mm to (176.7, 107.4), turned to 180 degrees
Routing:
- net VCC: track 25.1 -> 120.4 mm, vias 0 -> 4
- net /ESP_CS: track 10.4 -> 92.0 mm, vias 1 -> 4
- net /ESP_RTS: track 16.1 -> 97.2 mm
- net /SCK: track 93.1 -> 14.9 mm, vias 2 -> 1
- net /MISO: track 87.7 -> 13.8 mm, vias 2 -> 1
- net /ESP_RESET: track 21.3 -> 87.4 mm, vias 2 -> 6
- net /ESP_RX: track 26.3 -> 89.5 mm, vias 1 -> 2
- net /ESP_GPIO0: track 79.6 -> 22.6 mm
- net GND: track 11.0 -> 67.7 mm, vias 0 -> 8
- net /ESP_TX: track 36.0 -> 88.6 mm, vias 3 -> 6
- net /ESP_BUSY: track 77.5 -> 57.2 mm, vias 4 -> 2
- net /IO25: track 0.00 -> 15.7 mm, vias 0 -> 2
- net +3V3: track 27.4 -> 38.9 mm, vias 0 -> 2
- net Net-(D3-Pad1): track 0.00 -> 4.65 mm
- net /MOSI: track 52.9 -> 50.0 mm, vias 0 -> 2
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- added copper zone on B.Cu, net GND
