File: BLE_WIFI_HID/BLE_WIFI_HID.sch (KiCad schematic (older format))
At the start: 22 parts, among them P1 CONN_01X07, P2 CONN_01X07, P3 PROGRAMMER SERIAL, P4 Battery, SW1 SW_Push, U1 ESP32-WROOM, U2 AP2112K-3.3TRG1, U3 MCP73831T-2ACI/OT

Commit message: WIFININA new
Parts:
- removed SW1: SW_Push, TIH:SW_B3U-1000P, symbol SW_Push
- added R8: 10K, symbol Device:R_Small
- C1, C2, C3, C4: symbol C_Small -> device:C_Small
- D1, D3: symbol LED -> device:LED
- D2: symbol D_Schottky -> device:D_Schottky
- P1, P2: symbol CONN_01X07 -> conn:CONN_01X07
- P3: symbol CONN_01X06 -> conn:CONN_01X06
- P4: symbol CONN_01X02 -> conn:CONN_01X02
- R1, R2, R3, R5, R6, R7: symbol R_Small -> device:R_Small
- R4: value 1k -> 10k; symbol R_Small -> device:R_Small
- U1: symbol ESP32-WROOM -> ESP32-footprints-Shem-Lib:ESP32-WROOM
- U2: symbol AP2112K-3.3TRG1 -> electroniccats:AP2112K-3.3TRG1
- U3: symbol MCP73831T-2ACI/OT -> MCP73831T-2ACI_OT:MCP73831T-2ACI_OT
Connections:
- net labels added: ESP_BUSY, ESP_CS, ESP_GPIO0, ESP_RESET, ESP_RTS, ESP_RX, ESP_TX, IO25
- net labels removed: CS, I2S_D1/X7, I2S_SCK, IO0_BOOT/DTR, IO13, RESET/RTS, RX_ESP32, SCL, TX_ESP32
- wire segments 83 -> 94
- no-connect marks 36 -> 22
Other:
- note added: "NOTA: A donde va\nvoltaje bateria"
- note added: "NOTA: REVISAR\nRESISTENCIA\nDE RESET"

Commit message: change headers expansion
Parts:
- removed P1, P2: CONN_01X07, Pin_Headers:Pin_Header_Straight_1x07_Pitch2.54mm, symbol conn:CONN_01X07
- removed R1, R2: 100k, Resistors_SMD:R_0805_HandSoldering, symbol device:R_Small
- added J? (x2): Conn_02x03_Odd_Even, symbol Connector_Generic:Conn_02x03_Odd_Even
- C1, C2, C3, C4: symbol device:C_Small -> BLE_WIFI_HID-rescue:C_Small-device
- D1, D3: symbol device:LED -> BLE_WIFI_HID-rescue:LED-device
- D2: symbol device:D_Schottky -> BLE_WIFI_HID-rescue:D_Schottky-device
- P3: symbol conn:CONN_01X06 -> BLE_WIFI_HID-rescue:CONN_01X06-conn
- P4: symbol conn:CONN_01X02 -> BLE_WIFI_HID-rescue:CONN_01X02-conn
- R3, R4, R5, R6, R7: symbol device:R_Small -> BLE_WIFI_HID-rescue:R_Small-device
- U1: symbol ESP32-footprints-Shem-Lib:ESP32-WROOM -> BLE_WIFI_HID-rescue:ESP32-WROOM-ESP32-footprints-Shem-Lib
- U3: symbol MCP73831T-2ACI_OT:MCP73831T-2ACI_OT -> BLE_WIFI_HID-rescue:MCP73831T-2ACI_OT-MCP73831T-2ACI_OT
Connections:
- net ESP_BUSY: now also J?.5 (Pin_5)
- net ESP_CS: now also J?.2 (Pin_2)
- net ESP_GPIO0: now also J?.4 (Pin_4)
- net ESP_RESET: now also J?.5 (Pin_5)
- net ESP_RTS: now also J?.6 (Pin_6)
- net ESP_RX: now also J?.3 (Pin_3)
- net ESP_TX: now also J?.4 (Pin_4)
- net GND: now also J?.1 (Pin_1)
- net MISO: now also J?.2 (Pin_2)
- net MOSI: now also J?.1 (Pin_1)
- net SCK: now also J?.3 (Pin_3)
- net VCC: now also J?.6 (Pin_6)
Other:
- note removed: "NOTA: A donde va\nvoltaje bateria"
- moved on the sheet: D1, R3

Commit message: update to v0.3 pcb
Parts:
- J1, J2: renamed from J?; footprint (none) -> Pines:62000621121
- R8: footprint (none) -> Resistors_SMD:R_0805_HandSoldering
Changed lines of the file:
@@
 F 0 "R8" H 3979 2441 50  0000 L CNN
 F 1 "10K" H 3979 2350 50  0000 L CNN
-F 2 "" H 3920 2395 50  0001 C CNN
+F 2 "Resistors_SMD:R_0805_HandSoldering" H 3920 2395 50  0001 C CNN
 F 3 "~" H 3920 2395 50  0001 C CNN
 	1    3920 2395
@@
 ESP_BUSY
 $Comp
-L Connector_Generic:Conn_02x03_Odd_Even J?
+L Connector_Generic:Conn_02x03_Odd_Even J1
 U 1 1 5C95FB74
 P 7875 1295
-F 0 "J?" H 7925 1612 50  0000 C CNN
+F 0 "J1" H 7925 1612 50  0000 C CNN
 F 1 "Conn_02x03_Odd_Even" H 7925 1521 50  0000 C CNN
-F 2 "" H 7875 1295 50  0001 C CNN
+F 2 "Pines:62000621121" H 7875 1295 50  0001 C CNN
 F 3 "~" H 7875 1295 50  0001 C CNN
 	1    7875 1295
@@
 $EndComp
 $Comp
-L Connector_Generic:Conn_02x03_Odd_Even J?
+L Connector_Generic:Conn_02x03_Odd_Even J2
 U 1 1 5C95FBFE
 P 9875 1305
-F 0 "J?" H 9925 1622 50  0000 C CNN
+F 0 "J2" H 9925 1622 50  0000 C CNN
 F 1 "Conn_02x03_Odd_Even" H 9925 1531 50  0000 C CNN
-F 2 "" H 9875 1305 50  0001 C CNN
+F 2 "Pines:62000621121" H 9875 1305 50  0001 C CNN
 F 3 "~" H 9875 1305 50  0001 C CNN
 	1    9875 1305

Commit message: update reset resistor ESP32
Parts:
- C1, C2, C3, C4: symbol BLE_WIFI_HID-rescue:C_Small-device -> BLE_WIFI_HID-rescue:C_Small-device-BLE_WIFI_HID-rescue
- D1, D3: symbol BLE_WIFI_HID-rescue:LED-device -> BLE_WIFI_HID-rescue:LED-device-BLE_WIFI_HID-rescue
- D2: symbol BLE_WIFI_HID-rescue:D_Schottky-device -> BLE_WIFI_HID-rescue:D_Schottky-device-BLE_WIFI_HID-rescue
- P3: symbol BLE_WIFI_HID-rescue:CONN_01X06-conn -> BLE_WIFI_HID-rescue:CONN_01X06-conn-BLE_WIFI_HID-rescue
- P4: symbol BLE_WIFI_HID-rescue:CONN_01X02-conn -> BLE_WIFI_HID-rescue:CONN_01X02-conn-BLE_WIFI_HID-rescue
- R3, R4, R5, R6, R7: symbol BLE_WIFI_HID-rescue:R_Small-device -> BLE_WIFI_HID-rescue:R_Small-device-BLE_WIFI_HID-rescue
- U1: symbol BLE_WIFI_HID-rescue:ESP32-WROOM-ESP32-footprints-Shem-Lib -> BLE_WIFI_HID-rescue:ESP32-WROOM-ESP32-footprints-Shem-Lib-BLE_WIFI_HID-rescue
- U3: symbol BLE_WIFI_HID-rescue:MCP73831T-2ACI_OT-MCP73831T-2ACI_OT -> BLE_WIFI_HID-rescue:MCP73831T-2ACI_OT-MCP73831T-2ACI_OT-BLE_WIFI_HID-rescue
Other:
- note removed: "NOTA: REVISAR\nRESISTENCIA\nDE RESET"
- moved on the sheet: C2, C3, D2, R5, U2

Commit message: re-routeo
Parts:
- C1, C2, C3, C4: symbol BLE_WIFI_HID-rescue:C_Small-device-BLE_WIFI_HID-rescue -> BLE_WIFI_HID-rescue:C_Small-device-BLE_WIFI_HID-rescue-BLE_WIFI_HID-rescue
- D1, D3: symbol BLE_WIFI_HID-rescue:LED-device-BLE_WIFI_HID-rescue -> BLE_WIFI_HID-rescue:LED-device-BLE_WIFI_HID-rescue-BLE_WIFI_HID-rescue
- D2: symbol BLE_WIFI_HID-rescue:D_Schottky-device-BLE_WIFI_HID-rescue -> BLE_WIFI_HID-rescue:D_Schottky-device-BLE_WIFI_HID-rescue-BLE_WIFI_HID-rescue
- P3: symbol BLE_WIFI_HID-rescue:CONN_01X06-conn-BLE_WIFI_HID-rescue -> BLE_WIFI_HID-rescue:CONN_01X06-conn-BLE_WIFI_HID-rescue-BLE_WIFI_HID-rescue
- P4: symbol BLE_WIFI_HID-rescue:CONN_01X02-conn-BLE_WIFI_HID-rescue -> BLE_WIFI_HID-rescue:CONN_01X02-conn-BLE_WIFI_HID-rescue-BLE_WIFI_HID-rescue
- R3, R4, R5, R6, R7: symbol BLE_WIFI_HID-rescue:R_Small-device-BLE_WIFI_HID-rescue -> BLE_WIFI_HID-rescue:R_Small-device-BLE_WIFI_HID-rescue-BLE_WIFI_HID-rescue
- U1: symbol BLE_WIFI_HID-rescue:ESP32-WROOM-ESP32-footprints-Shem-Lib-BLE_WIFI_HID-rescue -> BLE_WIFI_HID-rescue:ESP32-WROOM-ESP32-footprints-Shem-Lib-BLE_WIFI_HID-rescue-BLE_WIFI_HID-rescue
- U2: symbol electroniccats:AP2112K-3.3TRG1 -> BLE_WIFI_HID-rescue:AP2112K-3.3TRG1-electroniccats
- U3: symbol BLE_WIFI_HID-rescue:MCP73831T-2ACI_OT-MCP73831T-2ACI_OT-BLE_WIFI_HID-rescue -> BLE_WIFI_HID-rescue:MCP73831T-2ACI_OT-MCP73831T-2ACI_OT-BLE_WIFI_HID-rescue-BLE_WIFI_HID-rescue
Changed lines of the file:
@@
 EESchema Schematic File Version 4
 LIBS:BLE_WIFI_HID-cache
-EELAYER 26 0
+EELAYER 29 0
 EELAYER END
 $Descr A4 11693 8268
@@
 $EndDescr
 $Comp
-L BLE_WIFI_HID-rescue:LED-device-BLE_WIFI_HID-rescue D1
+L BLE_WIFI_HID-rescue:LED-device-BLE_WIFI_HID-rescue-BLE_WIFI_HID-rescue D1
 U 1 1 5B26D928
 P 5655 1165
@@
 $EndComp
 $Comp
-L BLE_WIFI_HID-rescue:R_Small-device-BLE_WIFI_HID-rescue R3
+L BLE_WIFI_HID-rescue:R_Small-device-BLE_WIFI_HID-rescue-BLE_WIFI_HID-rescue R3
 U 1 1 5B26D96F
 P 5995 1165
@@
 $EndComp
 $Comp
-L BLE_WIFI_HID-rescue:R_Small-device-BLE_WIFI_HID-rescue R6
+L BLE_WIFI_HID-rescue:R_Small-device-BLE_WIFI_HID-rescue-BLE_WIFI_HID-rescue R6
 U 1 1 5B26D9F4
 P 4170 6940
@@
 $EndComp
 $Comp
-L BLE_WIFI_HID-rescue:R_Small-device-BLE_WIFI_HID-rescue R7
+L BLE_WIFI_HID-rescue:R_Small-device-BLE_WIFI_HID-rescue-BLE_WIFI_HID-rescue R7
 U 1 1 5B26DA52
 P 1670 7140
@@
 $EndComp
 $Comp
-L BLE_WIFI_HID-rescue:LED-device-BLE_WIFI_HID-rescue D3
+L BLE_WIFI_HID-rescue:LED-device-BLE_WIFI_HID-rescue-BLE_WIFI_HID-rescue D3
 U 1 1 5B26DBDC
 P 3860 6940
@@
 $EndComp
 $Comp
-L BLE_WIFI_HID-rescue:C_Small-device-BLE_WIFI_HID-rescue C4
+L BLE_WIFI_HID-rescue:C_Small-device-BLE_WIFI_HID-rescue-BLE_WIFI_HID-rescue C4
 U 1 1 5B26DC6D
 P 3495 7315
@@
 $EndComp
 $Comp
-L BLE_WIFI_HID-rescue:C_Small-device-BLE_WIFI_HID-rescue C1
+L BLE_WIFI_HID-rescue:C_Small-device-BLE_WIFI_HID-rescue-BLE_WIFI_HID-rescue C1
 U 1 1 5B26DCD8
 P 4505 1290
@@
 $EndComp
 $Comp
-L BLE_WIFI_HID-rescue:CONN_01X02-conn-BLE_WIFI_HID-rescue P4
+L BLE_WIFI_HID-rescue:CONN_01X02-conn-BLE_WIFI_HID-rescue-BLE_WIFI_HID-rescue P4
 U 1 1 5B26DD5E
 P 5190 7060
@@
 $EndComp
 $Comp
-L BLE_WIFI_HID-rescue:MCP73831T-2ACI_OT-MCP73831T-2ACI_OT-BLE_WIFI_HID-rescue U3
+L BLE_WIFI_HID-rescue:MCP73831T-2ACI_OT-MCP73831T-2ACI_OT-BLE_WIFI_HID-rescue-BLE_WIFI_HID-rescue U3
 U 1 1 5B26DF66
 P 2660 7040
@@
 $EndComp
 $Comp
-L BLE_WIFI_HID-rescue:+BATT-power1-BLE_WIFI_HID-rescue #PWR01
+L BLE_WIFI_HID-rescue:+BATT-power1-BLE_WIFI_HID-rescue-BLE_WIFI_HID-rescue #PWR01
 U 1 1 5B26EC4D
 P 3605 7125
@@
 $EndComp
 $Comp
-L BLE_WIFI_HID-rescue:GND-power1-BLE_WIFI_HID-rescue #PWR02
+L BLE_WIFI_HID-rescue:GND-power1-BLE_WIFI_HID-rescue-BLE_WIFI_HID-rescue #PWR02
 U 1 1 5B26EE21
 P 3495 7500
@@
 $EndComp
 $Comp
-L BLE_WIFI_HID-rescue:GND-power1-BLE_WIFI_HID-rescue #PWR03
+L BLE_WIFI_HID-rescue:GND-power1-BLE_WIFI_HID-rescue-BLE_WIFI_HID-rescue #PWR03
 U 1 1 5B26F0CC
 P 4890 7110
@@
 $EndComp
 $Comp
-L BLE_WIFI_HID-rescue:+BATT-power1-BLE_WIFI_HID-rescue #PWR04
+L BLE_WIFI_HID-rescue:+BATT-power1-BLE_WIFI_HID-rescue-BLE_WIFI_HID-rescue #PWR04
 U 1 1 5B26F118
 P 4885 7010
@@
 $EndComp
 $Comp
-L BLE_WIFI_HID-rescue:GND-power1-BLE_WIFI_HID-rescue #PWR05
+L BLE_WIFI_HID-rescue:GND-power1-BLE_WIFI_HID-rescue-BLE_WIFI_HID-rescue #PWR05
 U 1 1 5B26F308
 P 1975 3560
@@
 $EndComp
 $Comp
-L BLE_WIFI_HID-rescue:+3.3V-power1-BLE_WIFI_HID-rescue #PWR06
+L BLE_WIFI_HID-rescue:+3.3V-power1-BLE_WIFI_HID-rescue-BLE_WIFI_HID-rescue #PWR06
 U 1 1 5B26F442
 P 1385 1845
@@
 $EndComp
 $Comp
-L BLE_WIFI_HID-rescue:+3.3V-power1-BLE_WIFI_HID-rescue #PWR07
+L BLE_WIFI_HID-rescue:+3.3V-power1-BLE_WIFI_HID-rescue-BLE_WIFI_HID-rescue #PWR07
 U 1 1 5B26FB52
 P 4505 1070
@@
 $EndComp
 $Comp
-L BLE_WIFI_HID-rescue:GND-power1-BLE_WIFI_HID-rescue #PWR010
+L BLE_WIFI_HID-rescue:GND-power1-BLE_WIFI_HID-rescue-BLE_WIFI_HID-rescue #PWR010
 U 1 1 5B2700B6
 P 4505 1500
@@
 $EndComp
 $Comp
-L BLE_WIFI_HID-rescue:GND-power1-BLE_WIFI_HID-rescue #PWR011
+L BLE_WIFI_HID-rescue:GND-power1-BLE_WIFI_HID-rescue-BLE_WIFI_HID-rescue #PWR011
 U 1 1 5B270277
 P 5350 1195
@@
 $EndComp
 $Comp
-L BLE_WIFI_HID-rescue:VCC-power1-BLE_WIFI_HID-rescue #PWR012
+L BLE_WIFI_HID-rescue:VCC-power1-BLE_WIFI_HID-rescue-BLE_WIFI_HID-rescue #PWR012
 U 1 1 5B270483
 P 1480 6865
@@
 $EndComp
 $Comp
-L BLE_WIFI_HID-rescue:VCC-power1-BLE_WIFI_HID-rescue #PWR013
+L BLE_WIFI_HID-rescue:VCC-power1-BLE_WIFI_HID-rescue-BLE_WIFI_HID-rescue #PWR013
 U 1 1 5B270999
 P 4340 6860
@@
 NoConn ~ 3325 2805
 $Comp
-L BLE_WIFI_HID-rescue:ESP32-WROOM-ESP32-footprints-Shem-Lib-BLE_WIFI_HID-rescue U1
+L BLE_WIFI_HID-rescue:ESP32-WROOM-ESP32-footprints-Shem-Lib-BLE_WIFI_HID-rescue-BLE_WIFI_HID-rescue U1
 U 1 1 5B27204D
 P 2425 2455
@@
 NoConn ~ 1475 3055
 $Comp
-L BLE_WIFI_HID-rescue:GND-power1-BLE_WIFI_HID-rescue #PWR014
+L BLE_WIFI_HID-rescue:GND-power1-BLE_WIFI_HID-rescue-BLE_WIFI_HID-rescue #PWR014
 U 1 1 5B273B64
 P 3425 3185
@@
 $EndComp
 $Comp
-L BLE_WIFI_HID-rescue:GND-power1-BLE_WIFI_HID-rescue #PWR015
+L BLE_WIFI_HID-rescue:GND-power1-BLE_WIFI_HID-rescue-BLE_WIFI_HID-rescue #PWR015
 U 1 1 5B273C2E
 P 1385 3250
@@
 ESP_CS
 $Comp
-L BLE_WIFI_HID-rescue:VCC-power1-BLE_WIFI_HID-rescue #PWR016
+L BLE_WIFI_HID-rescue:VCC-power1-BLE_WIFI_HID-rescue-BLE_WIFI_HID-rescue #PWR016
 U 1 1 5B2759A9
 P 8875 1320
@@
 $EndComp
 $Comp
-L BLE_WIFI_HID-rescue:GND-power1-BLE_WIFI_HID-rescue #PWR017
+L BLE_WIFI_HID-rescue:GND-power1-BLE_WIFI_HID-rescue-BLE_WIFI_HID-rescue #PWR017
 U 1 1 5B2759F9
 P 9385 1020
@@
 $EndComp
 $Comp
-L BLE_WIFI_HID-rescue:CONN_01X06-conn-BLE_WIFI_HID-rescue P3
+L BLE_WIFI_HID-rescue:CONN_01X06-conn-BLE_WIFI_HID-rescue-BLE_WIFI_HID-rescue P3
 U 1 1 5B27613B
 P 9595 2805
@@
 ESP_RX
 $Comp
-L BLE_WIFI_HID-rescue:GND-power1-BLE_WIFI_HID-rescue #PWR018
+L BLE_WIFI_HID-rescue:GND-power1-BLE_WIFI_HID-rescue-BLE_WIFI_HID-rescue #PWR018
 U 1 1 5B276759
 P 9295 3055
@@
 REGULATOR
 $Comp
-L BLE_WIFI_HID-rescue:C_Small-device-BLE_WIFI_HID-rescue C2
+L BLE_WIFI_HID-rescue:C_Small-device-BLE_WIFI_HID-rescue-BLE_WIFI_HID-rescue C2
 U 1 1 5B27A891
 P 8135 5230
@@
 $EndComp
 $Comp
-L BLE_WIFI_HID-rescue:C_Small-device-BLE_WIFI_HID-rescue C3
+L BLE_WIFI_HID-rescue:C_Small-device-BLE_WIFI_HID-rescue-BLE_WIFI_HID-rescue C3
 U 1 1 5B27A920
 P 9645 5230
@@
 $EndComp
 $Comp
-L electroniccats:AP2112K-3.3TRG1 U2
+L BLE_WIFI_HID-rescue:AP2112K-3.3TRG1-electroniccats U2
 U 1 1 5B31ADE6
 P 9065 5275
@@
 $EndComp
 $Comp
-L BLE_WIFI_HID-rescue:R_Small-device-BLE_WIFI_HID-rescue R5
+L BLE_WIFI_HID-rescue:R_Small-device-BLE_WIFI_HID-rescue-BLE_WIFI_HID-rescue R5
 U 1 1 5B31B540
 P 8405 5275
@@
 $EndComp
 $Comp
-L BLE_WIFI_HID-rescue:GND-power1-BLE_WIFI_HID-rescue #PWR019
+L BLE_WIFI_HID-rescue:GND-power1-BLE_WIFI_HID-rescue-BLE_WIFI_HID-rescue #PWR019
 U 1 1 5B31BEE1
 P 8135 5380
@@
 $EndComp
 $Comp
-L BLE_WIFI_HID-rescue:D_Schottky-device-BLE_WIFI_HID-rescue D2
+L BLE_WIFI_HID-rescue:D_Schottky-device-BLE_WIFI_HID-rescue-BLE_WIFI_HID-rescue D2
 U 1 1 5B31BFE5
 P 8035 4870
@@
 $EndComp
 $Comp
-L BLE_WIFI_HID-rescue:+BATT-power1-BLE_WIFI_HID-rescue #PWR020
+L BLE_WIFI_HID-rescue:+BATT-power1-BLE_WIFI_HID-rescue-BLE_WIFI_HID-rescue #PWR020
 U 1 1 5B31C231
 P 8035 4695
@@
 $EndComp
 $Comp
-L BLE_WIFI_HID-rescue:VCC-power1-BLE_WIFI_HID-rescue #PWR021
+L BLE_WIFI_HID-rescue:VCC-power1-BLE_WIFI_HID-rescue-BLE_WIFI_HID-rescue #PWR021
 U 1 1 5B31C299
 P 7910 4700
@@
 $EndComp
 $Comp
-L BLE_WIFI_HID-rescue:+3.3V-power1-BLE_WIFI_HID-rescue #PWR022
+L BLE_WIFI_HID-rescue:+3.3V-power1-BLE_WIFI_HID-rescue-BLE_WIFI_HID-rescue #PWR022
 U 1 1 5B31C6F9
 P 9905 5055
@@
 $EndComp
 $Comp
-L BLE_WIFI_HID-rescue:GND-power1-BLE_WIFI_HID-rescue #PWR023
+L BLE_WIFI_HID-rescue:GND-power1-BLE_WIFI_HID-rescue-BLE_WIFI_HID-rescue #PWR023
 U 1 1 5B31C8E7
 P 9645 5580
@@
 ESP_GPIO0
 $Comp
-L BLE_WIFI_HID-rescue:VCC-power1-BLE_WIFI_HID-rescue #PWR024
+L BLE_WIFI_HID-rescue:VCC-power1-BLE_WIFI_HID-rescue-BLE_WIFI_HID-rescue #PWR024
 U 1 1 5B31D988
 P 8660 2765
@@
 ESP_RESET
 $Comp
-L BLE_WIFI_HID-rescue:R_Small-device-BLE_WIFI_HID-rescue R4
+L BLE_WIFI_HID-rescue:R_Small-device-BLE_WIFI_HID-rescue-BLE_WIFI_HID-rescue R4
 U 1 1 5B31E957
 P 1305 2055
